File: 1400-PSU/1400-PSU.kicad_pcb (KiCad board)
At the start: 2 copper layers, 173.4 x 62.1 mm, 50 parts, among them J1 Battery, J2 Jack-DC, J3 MAINBOARD_OUT, Q1 IRF9540N, SW1 SW_DPST, U1 MC34063, U2 MEZD41502A-C, U3 MEZD72401A-G, U4 LM340T-12, U5 N7812-1PH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

Commit message: resolve #6
Parts:
- added D5: 1N5819, Diode_THT:D_DO-41_SOD81_P10.16mm_Horizontal, F.Cu at (166.0, 78.0)
Connections:
- JP2 pad 2: Net-(A1-VIN) -> Net-(D5-A)
Routing:
- net Net-(A1-VIN): track 44.3 -> 24.5 mm, vias 1 -> 0
- net Net-(D5-A): track 0.00 -> 7.38 mm
