File: 1400-PSU/1400-PSU.kicad_sch (KiCad schematic)
At the start: 48 parts, among them J1 Battery, J2 Jack-DC, J3 MAINBOARD_OUT, Q1 IRF9540N, SW1 SW_DPST, U1 MC34063, U2 MEZD41502A-C, U3 MEZD72401A-G, U4 LM340T-12, U5 N7812-1PH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

Commit message: Minor updates, still need to figure out the charging issue and move the 15v converter down.
Parts:
- R4: value 20k -> 15k
Other:
- moved on the sheet: D4
Changed lines of the file:
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@@
 	(wire
 		(pts
-			(xy 97.79 24.13) (xy 100.33 24.13)
+			(xy 93.98 24.13) (xy 96.52 24.13)
 		)
 		(stroke
@@
 	(wire
 		(pts
-			(xy 107.95 24.13) (xy 109.22 24.13)
+			(xy 104.14 24.13) (xy 109.22 24.13)
 		)
 		(stroke
@@
 	(global_label "BATT_POS"
 		(shape input)
-		(at 97.79 24.13 180)
+		(at 93.98 24.13 180)
 		(fields_autoplaced yes)
 		(effects
@@
 		)
 		(property "Intersheetrefs" "${INTERSHEET_REFS}"
-			(at 85.7334 24.13 0)
+			(at 81.9234 24.13 0)
 			(effects
 				(font
@@
 		(length 2.54)
 		(shape round)
-		(at 107.95 24.13 0)
-		(fields_autoplaced yes)
+		(at 106.68 24.13 0)
 		(effects
 			(font
@@
 		)
 		(property "Netclass" "HI_POWER"
-			(at 108.6485 21.59 0)
+			(at 108.458 22.86 90)
 			(effects
 				(font
@@
 			)
 		)
-		(property "Value" "20k"
+		(property "Value" "15k"
 			(at 250.19 67.3099 0)
 			(effects
@@
 		(on_board yes)
 		(dnp no)
-		(fields_autoplaced yes)
 		(property "Reference" "#PWR014"
 			(at 132.08 35.56 0)
@@
 		)
 		(property "Value" "GND"
-			(at 132.08 34.29 0)
+			(at 134.62 32.512 0)
 			(effects
 				(font
@@
 		)
 		(property "Value" "MEZD41502A-C"
-			(at 129.032 36.83 0)
+			(at 129.032 35.814 0)
 			(effects
 				(font
@@
 	(symbol
 		(lib_id "Diode:1N4001")
-		(at 104.14 24.13 0)
+		(at 100.33 24.13 0)
 		(unit 1)
 		(exclude_from_sim no)
@@
 		(fields_autoplaced yes)
 		(property "Reference" "D4"
-			(at 104.14 17.78 0)
+			(at 100.33 17.78 0)
 			(effects
 				(font
@@
 		)
 		(property "Value" "31DQ06"
-			(at 104.14 20.32 0)
+			(at 100.33 20.32 0)
 			(effects
 				(font
@@
 		)
 		(property "Footprint" "Diode_THT:D_DO-201AD_P12.70mm_Horizontal"
-			(at 104.14 24.13 0)
+			(at 100.33 24.13 0)
 			(effects
 				(font
@@
 		)
 		(property "Datasheet" ""
-			(at 104.14 24.13 0)
+			(at 100.33 24.13 0)
 			(effects
 				(font
@@
 		)
 		(property "Description" ""
-			(at 104.14 24.13 0)
+			(at 100.33 24.13 0)
 			(effects
 				(font
@@
 		)
 		(property "Sim.Device" "D"
-			(at 104.14 24.13 0)
+			(at 100.33 24.13 0)
 			(effects
 				(font
@@
 		)
 		(property "Sim.Pins" "1=K 2=A"
-			(at 104.14 24.13 0)
+			(at 100.33 24.13 0)
 			(effects
 				(font

Commit message: Minor revisions.
Parts:
- added C10: 330uF 25V, Capacitor_THT:CP_Radial_D8.0mm_P5.00mm, symbol Device:C_Polarized
- J1: footprint Connector_JST:JST_EH_B2B-EH-A_1x02_P2.50mm_Vertical -> Connector_Wire:SolderWire-1.5sqmm_1x02_P7.8mm_D1.7mm_OD3.9mm
- J2: symbol Connector:Jack-DC -> Connector:Barrel_Jack_MountingPin
Connections:
- net GND: now also J2.MP (MountPin), C10.2
- net POWER_BRICK: now also C10.1
- net at D1.1 (K), D2.1 (K), JP2.3 (B): now also SW1.2, SW1.4; no longer SW1.1, SW1.3
- net at JP2.1 (A), U2.1 (VIN), U2.2 (VIN): now also SW1.1, SW1.3; no longer SW1.2, SW1.4
Other:
- moved on the sheet: SW1

Commit message: Adjust battery warning voltage dividers.
Parts:
- R5, R8: value 10k -> 200k
Changed lines of the file:
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@@
 			)
 		)
-		(property "Value" "10k"
+		(property "Value" "200k"
 			(at 161.29 81.2799 0)
 			(effects
@@
 			)
 		)
-		(property "Value" "10k"
+		(property "Value" "200k"
 			(at 170.18 96.5199 0)
 			(effects

Commit message: Minor update and fixes.
Parts:
- C2: value 47uF 50V -> 100uF 50V
Changed lines of the file:
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@@
 			)
 		)
-		(property "Value" "47uF 50V"
+		(property "Value" "100uF 50V"
 			(at 171.831 35.56 90)
 			(effects

Commit message: resolve #6
Parts:
- added D5: 1N5819, Diode_THT:D_DO-41_SOD81_P10.16mm_Horizontal, symbol Diode:1N5819
Connections:
- net at A1.30 (VIN): now also D5.1 (K); no longer JP2.2 (C)
- new net: D5.2 (A), JP2.2 (C)
Changed lines of the file:
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@@
 	(wire
 		(pts
-			(xy 129.54 80.01) (xy 97.79 80.01)
+			(xy 129.54 80.01) (xy 116.84 80.01)
 		)
 		(stroke
@@
 	(wire
 		(pts
+			(xy 109.22 80.01) (xy 97.79 80.01)
+		)
+		(stroke
+			(width 0)
+			(type default)
+		)
+	)
+	(wire
+		(pts
 			(xy 24.13 82.55) (xy 29.21 82.55)
 		)
@@
 		(length 2.54)
 		(shape round)
+		(at 120.65 80.01 0)
+		(fields_autoplaced yes)
+		(effects
+			(font
+				(size 1.27 1.27)
+			)
+			(justify left bottom)
+		)
+		(property "Netclass" "MED_POWER"
+			(at 121.3485 77.47 0)
+			(effects
+				(font
+					(size 1.27 1.27)
+					(italic yes)
+				)
+				(justify left)
+			)
+		)
+	)
+	(netclass_flag ""
+		(length 2.54)
+		(shape round)
 		(at 27.94 38.1 180)
 		(fields_autoplaced yes)
@@
 					(unit 1)
 				)
+			)
+		)
+	)
+	(symbol
+		(lib_id "Diode:1N5819")
+		(at 113.03 80.01 180)
+		(unit 1)
+		(exclude_from_sim no)
+		(in_bom yes)
+		(on_board yes)
+		(dnp no)
+		(fields_autoplaced yes)
+		(property "Reference" "D5"
+			(at 113.3475 73.66 0)
+			(effects
+				(font
+					(size 1.27 1.27)
+				)
+			)
+		)
+		(property "Value" "1N5819"
+			(at 113.3475 76.2 0)
+			(effects
+				(font
+					(size 1.27 1.27)
+				)
+			)
+		)
+		(property "Footprint" "Diode_THT:D_DO-41_SOD81_P10.16mm_Horizontal"
+			(at 113.03 75.565 0)
+			(effects
+				(font
+					(size 1.27 1.27)
+				)
+				(hide yes)
+			)
+		)
+		(property "Datasheet" "http://www.vishay.com/docs/88525/1n5817.pdf"
+			(at 113.03 80.01 0)
+			(effects
+				(font
+					(size 1.27 1.27)
+				)
+				(hide yes)
+			)
+		)
+		(property "Description" "40V 1A Schottky Barrier Rectifier Diode, DO-41"
+			(at 113.03 80.01 0)
+			(effects
+				(font
+					(size 1.27 1.27)
+				)
+				(hide yes)
+			)
+		)
+		(pin "2"
+		)
+		(pin "1"
+		)
+		(instances
+			(project "1400-PSU"
+				(path "/1e170452-a7b5-4944-9251-2ce18f45a364"
+					(reference "D5")
+					(unit 1)
+				)
